File: keyboard/keyboard.kicad_pcb (KiCad board)
At the start: 2 copper layers, 308.9 x 101.5 mm, 129 parts, among them J1 USB_C_Receptacle_USB2.0, J2 Programmer 1 time, J3 Addon interface, J4 Digital NOB, Q1 PMOS, U1 ATmega32U4-M, Y1 7F16000E09UCG

Commit message: battery connectors with diodes. (Should be replaced to FETs before production)
Parts:
- removed Q1: PMOS, Package_TO_SOT_SMD:TO-252-2
- removed R10: R100K, Resistor_SMD:R_0402_1005Metric
- added BT1: Battery, Connector_PinHeader_2.54mm:PinHeader_1x02_P2.54mm_Vertical, F.Cu at (152.8, 44.0)
- added D5: D, Diode_SMD:D_0402_1005Metric, B.Cu at (148.5, 44.6)
- added D6: D, Diode_SMD:D_0402_1005Metric, B.Cu at (148.5, 43.5)
- added SW1: SW_DIP_x01, Connector_PinHeader_2.54mm:PinHeader_1x02_P2.54mm_Vertical, F.Cu at (144.3, 44.0)
- D4: value 5V Zener -> D; footprint Diode_SMD:D_SOD-523 -> Diode_SMD:D_0402_1005Metric
- moved D4 40.1 mm to (148.6, 45.8), turned to 0 degrees
Connections:
- D4 pad 2: Net-(D4-A) -> /VIN
- J1 pad A4: /POWER_IN -> /VIN
- J1 pad A9: /POWER_IN -> /VIN
- J1 pad B4: /POWER_IN -> /VIN
- J1 pad B9: /POWER_IN -> /VIN
Routing:
- net /VIN: track 0.00 -> 39.4 mm, vias 0 -> 3
- net /VCC: track 709.3 -> 732.0 mm, vias 17 -> 18
- net /POWER_IN: track 22.5 -> 0.00 mm, vias 3 -> 0
- net Net-(D4-A): track 9.18 -> 0.00 mm
- net Net-(BT1-+): track 0.00 -> 8.12 mm
- net /VSWD: track 0.00 -> 3.99 mm
- net /GND: track 84.0 -> 82.3 mm

Commit message: Remove unnecessary files and add pullups for arrow keys.
Parts:
- added C24: 220pF, Capacitor_SMD:C_0402_1005Metric, B.Cu at (296.6, 120.8)
- added C25: 220pF, Capacitor_SMD:C_0402_1005Metric, B.Cu at (296.6, 121.8)
- added C26: 220pF, Capacitor_SMD:C_0402_1005Metric, B.Cu at (296.6, 122.8)
- added C27: 220pF, Capacitor_SMD:C_0402_1005Metric, B.Cu at (296.6, 123.8)
- added R10: R10K, Resistor_SMD:R_0402_1005Metric, B.Cu at (293.7, 120.8)
- added R21: R10K, Resistor_SMD:R_0402_1005Metric, B.Cu at (293.7, 121.8)
- added R22: R10K, Resistor_SMD:R_0402_1005Metric, B.Cu at (293.7, 122.8)
- added R23: R10K, Resistor_SMD:R_0402_1005Metric, B.Cu at (293.7, 123.8)
Routing:
- net /VCC: track 732.0 -> 755.9 mm, vias 18 -> 19
- net /KEY_66_ARR_RIGHT: track 144.4 -> 168.2 mm, vias 1 -> 2
- net /KEY_64_ARR_LEFT: track 102.2 -> 122.1 mm, vias 1 -> 2
- net /KEY_63_ARR_UP: track 125.9 -> 140.4 mm, vias 1 -> 2
- net /KEY_65_ARR_DOWN: track 124.1 -> 133.5 mm, vias 1 -> 2
- net /GND: vias 61 -> 60
