File: keyboard/keyboard.kicad_pcb (KiCad board)
At the start: 2 copper layers, 308.9 x 101.5 mm, 172 parts, among them J1 USB_C_Receptacle_USB2.0, J2 Programmer 1 time, J3 Addon interface, J4 Digital NOB, J5 USB_C1_USB2.0, J6 USB_A1, J7 USB_A2, U1 ATmega32U4-M, U2 USB2514-HZH (C184347), U3 TPS62140, U4 TPS2069C, U5 TPS2069C, U6 TPS2069C, Y1 16mhz, Y2 48mhz

Commit message: shematic and pcb update
Parts:
- removed C31, C32: 22pF, Capacitor_SMD:C_0402_1005Metric
- removed C33, C34: 1uF, Capacitor_SMD:C_0402_1005Metric
- removed J5: USB_C1_USB2.0, Connector_USB:USB_C_Receptacle_G-Switch_GT-USB-7010ASV
- removed J6: USB_A1, NORMAL_USB_A:GT_USBA
- removed J7: USB_A2, NORMAL_USB_A:GT_USBA
- removed L1: 2.2uH, Inductor_SMD:L_0805_2012Metric
- removed R24: R100K, Resistor_SMD:R_0402_1005Metric
- removed R25: R12K, Resistor_SMD:R_0402_1005Metric
- removed R26, R27, R28, R29, R30, R31: R10K, Resistor_SMD:R_0402_1005Metric
- removed R32, R41, R42: R1M, Resistor_SMD:R_0603_1608Metric
- removed R33, R34, R37, R38, R39, R40, R43, R44: R22, Resistor_SMD:R_0402_1005Metric
- removed R35, R36: 5.11K, Resistor_SMD:R_0402_1005Metric
- removed U4, U5, U6: TPS2069C, Package_TO_SOT_SMD:SOT-23-5
- removed Y2: 48mhz, Crystal:Crystal_SMD_TXC_7M-4Pin_3.2x2.5mm
- added BT1: Battery, Connector_PinHeader_2.54mm:PinHeader_1x02_P2.54mm_Vertical, F.Cu at (98.2, -1.70)
- added D5: D, Diode_SMD:D_0402_1005Metric, F.Cu at (106.8, -7.03)
- added D6: D, Diode_SMD:D_0402_1005Metric, F.Cu at (106.8, -5.04)
- added SW1: SW_DIP_x01, Connector_PinHeader_2.54mm:PinHeader_1x02_P2.54mm_Vertical, F.Cu at (102.8, -1.70)
- C2, C3: value 22pF -> 2pF
- U2: footprint Package_DFN_QFN:VQFN-48-1EP_7x7mm_P0.5mm_EP4.1x4.1mm_ThermalVias -> Package_DFN_QFN:VQFN-48-1EP_7x7mm_P0.5mm_EP4.1x4.1mm; moved to F.Cu
- Y1: value 16mhz -> 7F16000E09UCG
- moved U2 94.3 mm to (100.5, -8.67), turned to 0 degrees
- moved D3 55.1 mm to (261.1, 44.2)
- moved R5 55.1 mm to (258.5, 44.9)
- moved U3 48.2 mm to (107.8, -10.7)
- moved D2 47.6 mm to (246.1, 44.2)
- moved R4 47.6 mm to (243.5, 44.9)
- moved J4 46.5 mm to (286.0, 44.3)
- moved R3 40.2 mm to (228.4, 44.9)
- moved D1 40.1 mm to (231.1, 44.2)
- moved C28 34.7 mm to (106.6, -3.04)
- moved C29 34.7 mm to (106.6, -1.07)
- moved C30 34.7 mm to (106.6, 0.90)
Connections:
- net ADDR_A0 renamed /ADDR_A0
- net ADDR_A1 renamed /ADDR_A1
- net ADDR_A2 renamed /ADDR_A2
- net BOARD_EN renamed /BOARD_EN
- net KEY_00 renamed /KEY_00_~
- net KEY_01 renamed /KEY_01_1
- net KEY_02 renamed /KEY_02_2
- net KEY_03 renamed /KEY_03_3
- net KEY_04 renamed /KEY_04_4
- net KEY_05 renamed /KEY_05_5
- net KEY_06 renamed /KEY_06_6
- net KEY_07 renamed /KEY_07_7
- net KEY_08 renamed /KEY_08_8
- net KEY_09 renamed /KEY_09_9
- net KEY_10 renamed /KEY_10_0
- net KEY_11 renamed /KEY_11_-
- net KEY_12 renamed /KEY_12_=
- net KEY_13 renamed /KEY_13_BS
- net KEY_14 renamed /KEY_14_TAB
- net KEY_15 renamed /KEY_15_Q
- net KEY_16 renamed /KEY_16_W
- net KEY_17 renamed /KEY_17_E
- net KEY_18 renamed /KEY_18_R
- net KEY_19 renamed /KEY_19_T
- net KEY_20 renamed /KEY_20_Y
- net KEY_21 renamed /KEY_21_U
- net KEY_22 renamed /KEY_22_I
- net KEY_23 renamed /KEY_23_O
- net KEY_24 renamed /KEY_24_P
- net KEY_25 renamed /KEY_25_{
- net KEY_26 renamed /KEY_26_}
- net KEY_27 renamed /KEY_27_\
- net KEY_29 renamed /KEY_29_A
- net KEY_30 renamed /KEY_30_S
- net KEY_31 renamed /KEY_31_D
- net KEY_32 renamed /KEY_32_F
- net KEY_33 renamed /KEY_33_G
- net KEY_34 renamed /KEY_34_H
- net KEY_35 renamed /KEY_35_J
- net KEY_36 renamed /KEY_36_K
- net KEY_37 renamed /KEY_37_L
- net KEY_38 renamed /KEY_38_;
- net KEY_39 renamed /KEY_39_'
- net KEY_40 renamed /KEY_40_ENTER
- net KEY_41 renamed /KEY_41_LSHIFT
- net KEY_42 renamed /KEY_42_Z
- net KEY_43 renamed /KEY_43_X
- net KEY_44 renamed /KEY_44_C
- net KEY_45 renamed /KEY_45_V
- net KEY_46 renamed /KEY_46_B
- net KEY_47 renamed /KEY_47_N
- net KEY_48 renamed /KEY_48_M
- net KEY_49 renamed /KEY_49_,
- net KEY_50 renamed /KEY_50_.
- net KEY_51 renamed /KEY_51_?
- net KEY_52 renamed /KEY_52_RSHIFT
- net KEY_53 renamed /KEY_53_LCTRL
- net KEY_54 renamed /KEY_54_LWIN
- net KEY_55 renamed /KEY_55_LALT
- net KEY_56 renamed /KEY_56_SPACE
- net KEY_57 renamed /KEY_57_RALT
- net KEY_58 renamed /KEY_58_RFN
- net KEY_59 renamed /KEY_59_PtrScr
- net KEY_60 renamed /KEY_60_DEL
- net KEY_61 renamed /KEY_61_HOME
- net KEY_62 renamed /KEY_62_END
- net KEY_63 renamed /KEY_63_ARR_UP
- net KEY_64 renamed /KEY_64_ARR_LEFT
- net KEY_65 renamed /KEY_65_ARR_DOWN
- net KEY_66 renamed /KEY_66_ARR_RIGHT
- net SEG0 renamed /SEG0
- net SEG1 renamed /SEG1
- net SEG2 renamed /SEG2
- net SEG3 renamed /SEG3
- net SEG4 renamed /SEG4
- net SEG5 renamed /SEG5
- net SEG6 renamed /SEG6
- net SEG7 renamed /SEG7
- C1 pad 2: GND -> /GND
- C10 pad 1: VCC -> /VCC
- C10 pad 2: GND -> /GND
- C11 pad 1: VCC -> /VCC
- C11 pad 2: GND -> /GND
- C12 pad 1: VCC -> /VCC
- C12 pad 2: GND -> /GND
- C13 pad 1: VCC -> /VCC
- C13 pad 2: GND -> /GND
- C14 pad 1: VCC -> /VCC
- C14 pad 2: GND -> /GND
- C15 pad 1: VCC -> /VCC
- C15 pad 2: GND -> /GND
- C16 pad 1: GND -> /GND
- C17 pad 1: GND -> /GND
- C18 pad 1: GND -> /GND
- C19 pad 1: GND -> /GND
- C2 pad 2: GND -> /GND
- C20 pad 1: GND -> /GND
- C21 pad 1: GND -> /GND
- C22 pad 1: GND -> /GND
- C23 pad 1: GND -> /GND
- C24 pad 1: GND -> /GND
- C25 pad 1: GND -> /GND
- C26 pad 1: GND -> /GND
- C27 pad 1: GND -> /GND
- C28 pad 1: VCC -> /Bettery management and USB hub/VCC
- C28 pad 2: GND -> /Bettery management and USB hub/GND
- C29 pad 2: GND -> /Bettery management and USB hub/GND
- C3 pad 2: GND -> /GND
- C30 pad 1: /USB hub/3V3VCC -> /Bettery management and USB hub/3V3VCC
- C30 pad 2: GND -> /Bettery management and USB hub/GND
- C4 pad 1: VCC -> /VCC
- C4 pad 2: GND -> /GND
- C5 pad 1: VCC -> /VCC
- C5 pad 2: GND -> /GND
- C6 pad 1: VCC -> /VCC
- C6 pad 2: GND -> /GND
- C7 pad 1: VCC -> /VCC
- C7 pad 2: GND -> /GND
- C8 pad 1: VCC -> /VCC
- C8 pad 2: GND -> /GND
- C9 pad 1: VCC -> /VCC
- C9 pad 2: GND -> /GND
- J1 pad A1: GND -> /GND
- J1 pad A12: GND -> /GND
- J1 pad B1: GND -> /GND
- J1 pad B12: GND -> /GND
- J2 pad 2: VCC -> /VCC
- J2 pad 5: RESET -> /RESET
- J2 pad 6: GND -> /GND
- J3 pad 1: GND -> /GND
- J3 pad 2: VCC -> /VCC
- J4 pad 1: GND -> /GND
- J4 pad 2: VCC -> /VCC
- MUX1 pad 10: GND -> /GND
- MUX1 pad 17: GND -> /GND
- MUX1 pad 2: VCC -> /VCC
- MUX1 pad 7: /Key multiplezers/KEY_28_CL -> /KEY_28_CL
- MUX1 pad 9: GND -> /GND
- MUX2 pad 10: GND -> /GND
- MUX2 pad 17: GND -> /GND
- MUX2 pad 2: VCC -> /VCC
- MUX2 pad 9: GND -> /GND
- MUX3 pad 10: GND -> /GND
- MUX3 pad 17: GND -> /GND
- MUX3 pad 2: VCC -> /VCC
- MUX3 pad 9: GND -> /GND
- MUX4 pad 10: GND -> /GND
- MUX4 pad 17: GND -> /GND
- MUX4 pad 2: VCC -> /VCC
- MUX4 pad 9: GND -> /GND
- MUX5 pad 10: GND -> /GND
- MUX5 pad 17: GND -> /GND
- MUX5 pad 2: VCC -> /VCC
- MUX5 pad 9: GND -> /GND
- MUX6 pad 10: GND -> /GND
- MUX6 pad 17: GND -> /GND
- MUX6 pad 2: VCC -> /VCC
- MUX6 pad 9: GND -> /GND
- MUX7 pad 10: GND -> /GND
- MUX7 pad 17: GND -> /GND
- MUX7 pad 2: VCC -> /VCC
- MUX7 pad 9: GND -> /GND
- MUX8 pad 10: GND -> /GND
- MUX8 pad 17: GND -> /GND
- MUX8 pad 2: VCC -> /VCC
- MUX8 pad 9: GND -> /GND
- R1 pad 2: GND -> /GND
- R10 pad 1: VCC -> /VCC
- R11 pad 1: VCC -> /VCC
- R12 pad 1: VCC -> /VCC
- R13 pad 1: VCC -> /VCC
- R14 pad 1: VCC -> /VCC
- R15 pad 1: VCC -> /VCC
- R16 pad 1: VCC -> /VCC
- R17 pad 1: VCC -> /VCC
- R18 pad 1: VCC -> /VCC
- R19 pad 1: VCC -> /VCC
- R2 pad 2: GND -> /GND
- R20 pad 1: VCC -> /VCC
- R21 pad 1: VCC -> /VCC
- R22 pad 1: VCC -> /VCC
- R23 pad 1: VCC -> /VCC
- R3 pad 1: GND -> /GND
- R4 pad 1: GND -> /GND
- R5 pad 1: GND -> /GND
- R6 pad 2: GND -> /GND
- R7 pad 2: USBIN_D- -> /USBIN_D-
- R8 pad 2: USBIN_D+ -> /USBIN_D+
- R9 pad 2: GND -> /GND
- S1 pad 1: GND -> /GND
- S10 pad 1: GND -> /GND
- S11 pad 1: GND -> /GND
- S12 pad 1: GND -> /GND
- S13 pad 1: GND -> /GND
- S14 pad 1: GND -> /GND
- S15 pad 1: GND -> /GND
- S16 pad 1: GND -> /GND
- S17 pad 1: GND -> /GND
- S18 pad 1: GND -> /GND
- S19 pad 1: GND -> /GND
- S2 pad 1: GND -> /GND
- S20 pad 1: GND -> /GND
- S21 pad 1: GND -> /GND
- S22 pad 1: GND -> /GND
- S23 pad 1: GND -> /GND
- S24 pad 1: GND -> /GND
- S25 pad 1: GND -> /GND
- S26 pad 1: GND -> /GND
- S27 pad 1: GND -> /GND
- S28 pad 1: GND -> /GND
- S29 pad 1: GND -> /GND
- S29 pad 2: /Keys/KEY_28_CL -> /KEY_28_CL
- S3 pad 1: GND -> /GND
- S30 pad 1: GND -> /GND
- S31 pad 1: GND -> /GND
- S32 pad 1: GND -> /GND
- S33 pad 1: GND -> /GND
- S34 pad 1: GND -> /GND
- S35 pad 1: GND -> /GND
- S36 pad 1: GND -> /GND
- S37 pad 1: GND -> /GND
- S38 pad 1: GND -> /GND
- S39 pad 1: GND -> /GND
- S4 pad 1: GND -> /GND
- S40 pad 1: GND -> /GND
- S41 pad 1: GND -> /GND
- S42 pad 1: GND -> /GND
- S43 pad 1: GND -> /GND
- S44 pad 1: GND -> /GND
- S45 pad 1: GND -> /GND
- S46 pad 1: GND -> /GND
- S47 pad 1: GND -> /GND
- S48 pad 1: GND -> /GND
- S49 pad 1: GND -> /GND
- S5 pad 1: GND -> /GND
- S50 pad 1: GND -> /GND
- S51 pad 1: GND -> /GND
- S52 pad 1: GND -> /GND
- S53 pad 1: GND -> /GND
- S54 pad 1: GND -> /GND
- S55 pad 1: GND -> /GND
- S56 pad 1: GND -> /GND
- S57 pad 1: GND -> /GND
- S58 pad 1: GND -> /GND
- S59 pad 1: GND -> /GND
- S6 pad 1: GND -> /GND
- S60 pad 1: GND -> /GND
- S61 pad 1: GND -> /GND
- S62 pad 1: GND -> /GND
- S63 pad 1: GND -> /GND
- S64 pad 1: GND -> /GND
- S65 pad 1: GND -> /GND
- S66 pad 1: GND -> /GND
- S67 pad 1: GND -> /GND
- S7 pad 1: GND -> /GND
- S8 pad 1: GND -> /GND
- S9 pad 1: GND -> /GND
- U1 pad 13: RESET -> /RESET
- U1 pad 14: VCC -> /VCC
- U1 pad 15: GND -> /GND
- U1 pad 2: VCC -> /VCC
- U1 pad 23: GND -> /GND
- U1 pad 24: VCC -> /VCC
- U1 pad 3: USBMCU_D- -> /USBMCU_D-
- U1 pad 34: VCC -> /VCC
- U1 pad 35: GND -> /GND
- U1 pad 4: USBMCU_D+ -> /USBMCU_D+
- U1 pad 42: GND -> /GND
- U1 pad 43: GND -> /GND
- U1 pad 44: VCC -> /VCC
- U1 pad 45: GND -> /GND
- U1 pad 5: GND -> /GND
- U1 pad 7: VCC -> /VCC
- U2 pad 1: Net-(U2-USBDM_DN1/PRT_DIS_M1) -> unconnected-(U2-USBDM_DN1/PRT_DIS_M1-Pad1)
- U2 pad 10: /USB hub/3V3VCC -> unconnected-(U2-VDDA33-Pad10)
- U2 pad 11: (no net) -> unconnected-(U2-TEST-Pad11)
- U2 pad 12: (no net) -> unconnected-(U2-PRTPWR1/BC_EN1-Pad12)
- U2 pad 17: Net-(U2-CRFILT) -> unconnected-(U2-OCS_N2-Pad17)
- U2 pad 18: /USB hub/3V3VCC -> unconnected-(U2-PRTPWR3/BC_EN3-Pad18)
- U2 pad 19: /USB hub/USBHUBC1_PWR -> unconnected-(U2-OCS_N3-Pad19)
- U2 pad 2: Net-(U2-USBDP_DN1/PRT_DIS_P1) -> unconnected-(U2-USBDP_DN1/PRT_DIS_P1-Pad2)
- U2 pad 20: /USB hub/USBHUBC1_~{OCS} -> unconnected-(U2-PRTPWR4/BC_EN4-Pad20)
- U2 pad 21: /USB hub/USBHUBA1_PWR -> unconnected-(U2-OCS_N4-Pad21)
- U2 pad 26: /USB hub/USBHUBA1_~{OCS} -> unconnected-(U2-RESET_N-Pad26)
- U2 pad 27: /USB hub/USBHUBA2_PWR -> unconnected-(U2-VBUS_DET-Pad27)
- U2 pad 28: /USB hub/USBHUBA2_~{OCS} -> unconnected-(U2-SUSP_IND/LOCAL_PWR/NON_REM0-Pad28)
- U2 pad 29: /USB hub/NON_REM1 -> unconnected-(U2-VDDA33-Pad29)
- U2 pad 3: /USB hub/USBHUBC1_D- -> unconnected-(U2-USBDM_DN2/PRT_DIS_M2-Pad3)
- U2 pad 30: /USB hub/3V3VCC -> /Bettery management and USB hub/USBIN_D-
- U2 pad 31: /USB hub/CFG_SEL0 -> /Bettery management and USB hub/USBIN_D+
- U2 pad 32: /USB hub/CFG_SEL1 -> unconnected-(U2-XTALOUT-Pad32)
- U2 pad 33: /USB hub/CFG_SEL2 -> unconnected-(U2-XTALIN/CLKIN-Pad33)
- U2 pad 34: RESET -> unconnected-(U2-PLLFILT-Pad34)
- U2 pad 35: /USB hub/3V3VCC -> unconnected-(U2-RBIAS-Pad35)
- U2 pad 38: /USB hub/3V3VCC -> (no net)
- U2 pad 39: /USB hub/NON_REM0 -> (no net)
- U2 pad 4: /USB hub/USBHUBC1_D+ -> unconnected-(U2-USBDP_DN2/PRT_DIS_P2-Pad4)
- U2 pad 40: /USB hub/SEL48 -> (no net)
- U2 pad 41: /USB hub/3V3VCC -> (no net)
- U2 pad 42: USBIN_D- -> (no net)
- U2 pad 43: USBIN_D+ -> (no net)
- U2 pad 44: Net-(U2-XTALOUT) -> (no net)
- U2 pad 45: Net-(U2-XTALIN/CLKIN) -> (no net)
- U2 pad 46: Net-(U2-PLLFILT) -> (no net)
- U2 pad 47: Net-(U2-RBIAS) -> (no net)
- U2 pad 48: /USB hub/3V3VCC -> (no net)
- U2 pad 49: GND -> (no net)
- U2 pad 5: /USB hub/3V3VCC -> unconnected-(U2-VDDA33-Pad5)
- U2 pad 6: /USB hub/USBHUBA1_D- -> unconnected-(U2-USBDM_DN3/PRT_DIS_M3-Pad6)
- U2 pad 7: /USB hub/USBHUBA1_D+ -> unconnected-(U2-USBDP_DN3/PRT_DIS_P3-Pad7)
- U2 pad 8: /USB hub/USBHUBA2_D- -> unconnected-(U2-USBDM_DN4/PRT_DIS_M4-Pad8)
- U2 pad 9: /USB hub/USBHUBA2_D+ -> unconnected-(U2-USBDP_DN4/PRT_DIS_P4-Pad9)
- U3 pad 10: VCC -> /Bettery management and USB hub/VCC
- U3 pad 11: VCC -> /Bettery management and USB hub/VCC
- U3 pad 12: VCC -> /Bettery management and USB hub/VCC
- U3 pad 13: VCC -> /Bettery management and USB hub/VCC
- U3 pad 14: /USB hub/3V3VCC -> /Bettery management and USB hub/3V3VCC
- U3 pad 15: GND -> /Bettery management and USB hub/GND
- U3 pad 16: GND -> /Bettery management and USB hub/GND
- U3 pad 17: GND -> /Bettery management and USB hub/GND
- U3 pad 5: GND -> /Bettery management and USB hub/GND
- U3 pad 6: GND -> /Bettery management and USB hub/GND
- U3 pad 7: GND -> /Bettery management and USB hub/GND
- U3 pad 8: GND -> /Bettery management and USB hub/GND
- Y1 pad 2: GND -> /GND
- Y1 pad 4: GND -> /GND
Routing:
- net VCC: track 760.8 -> 0.00 mm, vias 17 -> 0
- net /VCC: track 0.00 -> 721.3 mm, vias 0 -> 17
- net (no net): track 27.6 -> 202.3 mm
- net GND: track 82.3 -> 0.00 mm, vias 58 -> 0
- net /GND: track 0.00 -> 82.3 mm, vias 0 -> 60
- net USBMCU_D+: track 76.9 -> 0.00 mm
- net USBMCU_D-: track 76.0 -> 0.00 mm
- net RESET: track 34.1 -> 0.00 mm, vias 1 -> 0
- net /RESET: track 0.00 -> 34.1 mm, vias 0 -> 1
- net /KEY_28_CL: track 0.00 -> 27.6 mm
- net /LED_2: track 154.0 -> 180.9 mm, vias 0 -> 1
- net /VNOB_A: track 215.2 -> 191.4 mm, vias 1 -> 0
- net /VNOB_B: track 219.8 -> 196.1 mm, vias 1 -> 0
- net /LED_1: track 155.3 -> 169.7 mm, vias 0 -> 1
- net /LED_0: track 156.7 -> 165.8 mm, vias 0 -> 1
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- added copper zone on B.Cu, net /GND
- added copper zone on F.Cu, net /GND
- removed copper zone on B.Cu, net GND
- removed copper zone on F.Cu, net GND
