File: keyboard/_autosave-keyboard.kicad_pcb (KiCad board)
At the start: 2 copper layers, 308.9 x 101.5 mm, 143 parts, among them J1 USB_C_Receptacle_USB2.0, J2 Programmer 1 time, J3 Addon interface, J4 Digital NOB, SW1 SW_DIP_x01, U1 ATmega32U4-M, U2 USB2514-HZH (C184347), U3 TPS62140, Y1 7F16000E09UCG

Commit message: wireing
Parts:
- U2: moved to B.Cu
- moved U2 106.5 mm to (180.8, 61.3), turned to 90 degrees
- moved BT1 50.8 mm to (139.9, 27.4)
- moved C28 50.8 mm to (148.3, 26.0)
- moved C29 50.8 mm to (148.3, 28.0)
- moved C30 50.8 mm to (148.3, 29.9)
- moved U3 50.8 mm to (149.5, 18.4)
- moved D5 50.8 mm to (148.5, 22.0)
- moved D6 50.8 mm to (148.5, 24.0)
- moved SW1 50.8 mm to (144.5, 27.4)
Connections:
- U2 pad 1: unconnected-(U2-USBDM_DN1/PRT_DIS_M1-Pad1) -> /Bettery management and USB hub/USBMCU_D-
- U2 pad 2: unconnected-(U2-USBDP_DN1/PRT_DIS_P1-Pad2) -> /Bettery management and USB hub/USBMCU_D+
