File: keyboard/keyboard.kicad_sch (KiCad schematic)
At the start: 135 parts, among them J1 USB_C_Receptacle_USB2.0, J2 Programmer 1 time, J3 Addon interface, J4 Digital NOB, U1 ATmega32U4-M, Y1 7F16000E09UCG

Commit message: wireing
Parts:
- removed D4: D, Diode_SMD:D_0402_1005Metric, symbol Device:D
- C2, C3: value 2pF -> 22pF
- Y1: value 7F16000E09UCG -> 16mhz
Connections:
- net USB_D+ renamed USBIN_D+
- net USBIN_D+: no longer U1.4 (D+)
- net USB_D- renamed USBIN_D-
- net USBIN_D-: no longer U1.3 (D-)
- new net USBMCU_D+: U1.4 (D+)
- new net USBMCU_D-: U1.3 (D-)
Other:
- moved on the sheet: R1, R2
Changed lines of the file:
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@@
   (junction (at 287.02 176.53) (diameter 0) (color 0 0 0 0)
   )
+  (junction (at 252.73 261.62) (diameter 0) (color 0 0 0 0)
+  )
   (junction (at 212.09 78.74) (diameter 0) (color 0 0 0 0)
   )
@@
   (junction (at 388.62 88.9) (diameter 0) (color 0 0 0 0)
   )
-  (junction (at 251.46 243.84) (diameter 0) (color 0 0 0 0)
-  )
   (junction (at 231.14 171.45) (diameter 0) (color 0 0 0 0)
   )
   (junction (at 19.05 121.92) (diameter 0) (color 0 0 0 0)
   )
-  (junction (at 251.46 261.62) (diameter 0) (color 0 0 0 0)
-  )
   (junction (at 105.41 226.06) (diameter 0) (color 0 0 0 0)
   )
@@
   (junction (at 208.28 69.85) (diameter 0) (color 0 0 0 0)
   )
+  (junction (at 252.73 243.84) (diameter 0) (color 0 0 0 0)
+  )
   (junction (at 260.35 78.74) (diameter 0) (color 0 0 0 0)
   )
@@
     (stroke (width 0) (type default))
   )
-  (wire (pts (xy 251.46 243.84) (xy 251.46 261.62))
+  (wire (pts (xy 252.73 243.84) (xy 252.73 261.62))
     (stroke (width 0) (type default))
   )
@@
     (stroke (width 0) (type default))
   )
-  (wire (pts (xy 251.46 261.62) (xy 261.62 261.62))
-    (stroke (width 0) (type default))
-  )
   (wire (pts (xy 86.36 162.56) (xy 100.33 162.56))
     (stroke (width 0) (type default))
@@
     (stroke (width 0) (type default))
   )
-  (wire (pts (xy 261.62 226.06) (xy 261.62 231.14))
+  (wire (pts (xy 262.89 226.06) (xy 262.89 231.14))
     (stroke (width 0) (type default))
   )
@@
     (stroke (width 0) (type default))
   )
-  (wire (pts (xy 226.06 226.06) (xy 261.62 226.06))
+  (wire (pts (xy 226.06 226.06) (xy 262.89 226.06))
     (stroke (width 0) (type default))
   )
@@
     (stroke (width 0) (type default))
   )
+  (wire (pts (xy 252.73 261.62) (xy 261.62 261.62))
+    (stroke (width 0) (type default))
+  )
   (wire (pts (xy 227.33 198.12) (xy 231.14 198.12))
     (stroke (width 0) (type default))
@@
     (stroke (width 0) (type default))
   )
-  (wire (pts (xy 331.47 189.23) (xy 341.63 189.23))
+  (wire (pts (xy 327.66 189.23) (xy 341.63 189.23))
     (stroke (width 0) (type default))
   )
@@
     (stroke (width 0) (type default))
   )
-  (wire (pts (xy 226.06 228.6) (xy 251.46 228.6))
+  (wire (pts (xy 226.06 228.6) (xy 252.73 228.6))
     (stroke (width 0) (type default))
   )
@@
     (stroke (width 0) (type default))
   )
-  (wire (pts (xy 251.46 228.6) (xy 251.46 231.14))
+  (wire (pts (xy 252.73 228.6) (xy 252.73 231.14))
     (stroke (width 0) (type default))
   )
@@
     (stroke (width 0) (type default))
   )
-  (wire (pts (xy 261.62 243.84) (xy 251.46 243.84))
+  (wire (pts (xy 262.89 243.84) (xy 252.73 243.84))
     (stroke (width 0) (type default))
   )
@@
     (stroke (width 0) (type default))
   )
-  (wire (pts (xy 261.62 238.76) (xy 261.62 243.84))
+  (wire (pts (xy 262.89 238.76) (xy 262.89 243.84))
     (stroke (width 0) (type default))
   )
@@
     (stroke (width 0) (type default))
   )
-  (wire (pts (xy 245.11 220.98) (xy 261.62 220.98))
-    (stroke (width 0) (type default))
-  )
   (wire (pts (xy 62.23 33.02) (xy 62.23 45.72))
     (stroke (width 0) (type default))
@@
     (stroke (width 0) (type default))
   )
-  (wire (pts (xy 251.46 238.76) (xy 251.46 243.84))
+  (wire (pts (xy 252.73 238.76) (xy 252.73 243.84))
     (stroke (width 0) (type default))
   )
@@
     (stroke (width 0) (type default))
   )
-  (wire (pts (xy 331.47 186.69) (xy 341.63 186.69))
+  (wire (pts (xy 327.66 186.69) (xy 341.63 186.69))
     (stroke (width 0) (type default))
   )
@@
     (stroke (width 0) (type default))
   )
-  (wire (pts (xy 215.9 261.62) (xy 251.46 261.62))
+  (wire (pts (xy 215.9 261.62) (xy 252.73 261.62))
     (stroke (width 0) (type default))
   )
@@
     (effects (font (size 1.27 1.27)) (justify left bottom))
   )
-  (label "USB_D-" (at 240.03 233.68 0) (fields_autoplaced)
+  (label "USBIN_D-" (at 240.03 233.68 0) (fields_autoplaced)
     (effects (font (size 1.27 1.27)) (justify left bottom))
   )
@@
     (effects (font (size 1.27 1.27)) (justify left bottom))
   )
-  (label "USB_D-" (at 331.47 189.23 0) (fields_autoplaced)
+  (label "USBMCU_D-" (at 327.66 189.23 0) (fields_autoplaced)
     (effects (font (size 1.27 1.27)) (justify left bottom))
   )
@@
     (effects (font (size 1.27 1.27)) (justify left bottom))
   )
-  (label "USB_D+" (at 331.47 186.69 0) (fields_autoplaced)
+  (label "USBMCU_D+" (at 327.66 186.69 0) (fields_autoplaced)
     (effects (font (size 1.27 1.27)) (justify left bottom))
   )
@@
     (effects (font (size 1.27 1.27)) (justify left bottom))
   )
-  (label "USB_D+" (at 240.03 238.76 0) (fields_autoplaced)
+  (label "USBIN_D+" (at 240.03 238.76 0) (fields_autoplaced)
     (effects (font (size 1.27 1.27)) (justify left bottom))
   )
@@
     (effects (font (size 1.27 1.27)) (justify left bottom))
   )
-  (label "VCC" (at 257.81 220.98 0) (fields_autoplaced)
-    (effects (font (size 1.27 1.27)) (justify left bottom))
-  )
   (label "GND" (at 314.96 209.55 0) (fields_autoplaced)
     (effects (font (size 1.27 1.27)) (justify left bottom))
@@
     )
   )
-  (symbol (lib_id "Device:R") (at 251.46 234.95 0) (unit 1)
+  (symbol (lib_id "Device:R") (at 252.73 234.95 0) (unit 1)
     (in_bom yes) (on_board yes) (dnp no) (fields_autoplaced)
-    (property "Reference" "R1" (at 254 233.68 0)
+    (property "Reference" "R1" (at 255.27 233.68 0)
       (effects (font (size 1.27 1.27)) (justify left))
     )
-    (property "Value" "5.11K" (at 254 236.22 0)
+    (property "Value" "5.11K" (at 255.27 236.22 0)
       (effects (font (size 1.27 1.27)) (justify left))
     )
-    (property "Footprint" "Resistor_SMD:R_0402_1005Metric" (at 249.682 234.95 90)
+    (property "Footprint" "Resistor_SMD:R_0402_1005Metric" (at 250.952 234.95 90)
       (effects (font (size 1.27 1.27)) hide)
     )
-    (property "Datasheet" "~" (at 251.46 234.95 0)
+    (property "Datasheet" "~" (at 252.73 234.95 0)
       (effects (font (size 1.27 1.27)) hide)
     )
@@
     )
   )
-  (symbol (lib_id "Device:D") (at 241.3 220.98 180) (unit 1)
-    (in_bom yes) (on_board yes) (dnp no)
-    (property "Reference" "D4" (at 241.3 217.17 0)
-      (effects (font (size 1.27 1.27)))
-    )
-    (property "Value" "D" (at 240.03 217.17 0)
-      (effects (font (size 1.27 1.27)) hide)
-    )
-    (property "Footprint" "Diode_SMD:D_0402_1005Metric" (at 241.3 220.98 0)
-      (effects (font (size 1.27 1.27)) hide)
-    )
-    (property "Datasheet" "~" (at 241.3 220.98 0)
-      (effects (font (size 1.27 1.27)) hide)
-    )
-    (property "Sim.Device" "D" (at 241.3 220.98 0)
-      (effects (font (size 1.27 1.27)) hide)
-    )
-    (property "Sim.Pins" "1=K 2=A" (at 241.3 220.98 0)
-      (effects (font (size 1.27 1.27)) hide)
-    )
-    (pin "1")
-    (pin "2")
-    (instances
-      (project "keyboard"
-        (path "/ba343d94-601d-44c5-b848-a7d9121c7be9"
-          (reference "D4") (unit 1)
-        )
-      )
-    )
-  )
   (symbol (lib_id "PG151101S11:PG151101S11") (at 76.2 276.86 0) (unit 1)
     (in_bom yes) (on_board yes) (dnp no) (fields_autoplaced)
@@
       (effects (font (size 1.27 1.27)))
     )
-    (property "Value" "7F16000E09UCG" (at 299.72 171.45 0)
+    (property "Value" "16mhz" (at 299.72 171.45 0)
       (effects (font (size 1.27 1.27)))
     )
@@
       (effects (font (size 1.27 1.27)) (justify left))
     )
-    (property "Value" "2pF" (at 290.83 182.88 0)
+    (property "Value" "22pF" (at 290.83 182.88 0)
       (effects (font (size 1.27 1.27)) (justify left))
     )
@@
     )
   )
-  (symbol (lib_id "Device:R") (at 261.62 234.95 0) (unit 1)
+  (symbol (lib_id "Device:R") (at 262.89 234.95 0) (unit 1)
     (in_bom yes) (on_board yes) (dnp no)
-    (property "Reference" "R2" (at 264.16 233.68 0)
+    (property "Reference" "R2" (at 265.43 233.68 0)
       (effects (font (size 1.27 1.27)) (justify left))
     )
-    (property "Value" "5.11K" (at 264.16 236.22 0)
+    (property "Value" "5.11K" (at 265.43 236.22 0)
       (effects (font (size 1.27 1.27)) (justify left))
     )
-    (property "Footprint" "Resistor_SMD:R_0402_1005Metric" (at 259.842 234.95 90)
+    (property "Footprint" "Resistor_SMD:R_0402_1005Metric" (at 261.112 234.95 90)
       (effects (font (size 1.27 1.27)) hide)
     )
-    (property "Datasheet" "~" (at 261.62 234.95 0)
+    (property "Datasheet" "~" (at 262.89 234.95 0)
       (effects (font (size 1.27 1.27)) hide)
     )
@@
       (effects (font (size 1.27 1.27)) (justify left))
     )
-    (property "Value" "2pF" (at 316.23 182.88 0)
+    (property "Value" "22pF" (at 316.23 182.88 0)
       (effects (font (size 1.27 1.27)) (justify left))
     )
