File: pcb/key_muxes.kicad_sch (KiCad schematic)
At the start: 40 parts

Commit message: new versions and finalized wired version
Connections:
- net KEY_11: now also MUX7.14 (Y3); no longer MUX7.15 (Y0)
- net KEY_25: now also MUX7.15 (Y0); no longer MUX7.14 (Y3)
Changed lines of the file:
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@@
+    (effects (font (size 1.27 1.27)) (justify left bottom))
+  )
+  (label "KEY_25_{" (at 153.67 57.15 0) (fields_autoplaced)
     (effects (font (size 1.27 1.27)) (justify left bottom))
   )
@@
     (effects (font (size 1.27 1.27)) (justify left bottom))
   )
-  (label "KEY_11_-" (at 153.67 57.15 0) (fields_autoplaced)
-    (effects (font (size 1.27 1.27)) (justify left bottom))
-  )
   (label "SEG3" (at 213.36 45.72 0) (fields_autoplaced)
     (effects (font (size 1.27 1.27)) (justify left bottom))
@@
   )
   (label "GND" (at 120.65 45.72 0) (fields_autoplaced)
+    (effects (font (size 1.27 1.27)) (justify left bottom))
+  )
+  (label "KEY_11_-" (at 153.67 64.77 0) (fields_autoplaced)
     (effects (font (size 1.27 1.27)) (justify left bottom))
   )
@@
     (effects (font (size 1.27 1.27)) (justify left bottom))
   )
-  (label "KEY_25_{" (at 153.67 64.77 0) (fields_autoplaced)
-    (effects (font (size 1.27 1.27)) (justify left bottom))
-  )
