File: pcb/keyboard.kicad_pcb (KiCad board)
At the start: 2 copper layers, 308.9 x 101.5 mm, 172 parts, among them J1 USB_C_Receptacle_USB2.0, J2 Programmer 1 time, J3 Addon interface, J4 Digital NOB, J5 USB_C1_USB2.0, J6 USB_A1, J7 USB_A2, U1 ATmega32U4-M, U2 USB2514-HZH (C184347), U3 TPS62140, U4 TPS2069C, U5 TPS2069C, U6 TPS2069C, Y1 16mhz, Y2 48mhz

Commit message: new versions and finalized wired version
Parts:
- C28, C29, C30, C31, C32, C33, C34, L1, R24, R25, R26, R27, R28, R29, R30, R31, R32, R33, R34, R35, R36, R37, R38, R39, R40, R41, R42, R43, R44, U3, U4, Y2: moved to B.Cu
- moved R42 158.8 mm to (299.2, 45.0), turned to 90 degrees
- moved R41 150.5 mm to (290.4, 45.0), turned to 90 degrees
- moved U4 130.7 mm to (256.7, 58.0), turned to 180 degrees
- moved R32 125.9 mm to (263.9, 48.4), turned to -90 degrees
- moved R35 121.2 mm to (258.9, 50.1), turned to -90 degrees
- moved R36 117.9 mm to (256.1, 50.2), turned to -90 degrees
- moved L1 81.1 mm to (159.6, 51.6), turned to -90 degrees
- moved R26 62.5 mm to (160.6, 57.1), turned to -90 degrees
- moved R27 61.6 mm to (155.7, 61.0)
- moved R28 60.7 mm to (155.7, 62.0)
- moved R29 59.9 mm to (155.7, 63.0)
- moved R39 59.6 mm to (170.1, 67.0)
- moved R30 59.0 mm to (155.7, 64.0)
- moved R38 58.6 mm to (170.1, 64.0)
- moved R33 57.6 mm to (170.1, 62.0)
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Connections:
- J1 pad A4: /VIN -> VCC
- J1 pad A9: /VIN -> VCC
- J1 pad B4: /VIN -> VCC
- J1 pad B9: /VIN -> VCC
- MUX7 pad 14: KEY_25 -> KEY_11
- MUX7 pad 15: KEY_11 -> KEY_25
- U1 pad 20: /LED_2 -> /LED_0
- U1 pad 22: /LED_0 -> /LED_2
Routing:
- net /USB hub/USBHUBA2_~{OCS}: track 0.00 -> 211.6 mm, vias 0 -> 2
- net /USB hub/USBHUBA2_PWR: track 0.00 -> 211.1 mm, vias 0 -> 2
- net /USB hub/USBHUBA1_~{OCS}: track 0.00 -> 169.3 mm, vias 0 -> 2
- net /USB hub/USBHUBA1_PWR: track 0.00 -> 166.7 mm, vias 0 -> 2
- net /USB hub/USBHUBC1_~{OCS}: track 0.00 -> 146.8 mm, vias 0 -> 2
- net Net-(J7-D+): track 0.00 -> 145.6 mm, vias 0 -> 2
- net /USB hub/USBHUBC1_PWR: track 0.00 -> 144.7 mm, vias 0 -> 2
- net Net-(J7-D-): track 0.00 -> 143.2 mm, vias 0 -> 2
- net Net-(J6-D+): track 0.00 -> 119.7 mm, vias 0 -> 2
- net RESET: track 34.1 -> 152.0 mm, vias 1 -> 3
- net Net-(J6-D-): track 0.00 -> 117.3 mm, vias 0 -> 2
- net Net-(J5-D+-PadA6): track 0.00 -> 99.7 mm, vias 0 -> 2
- net Net-(J5-D--PadA7): track 0.00 -> 99.5 mm, vias 0 -> 2
- net /LED_2: track 154.0 -> 218.0 mm, vias 0 -> 1
- net /LED_1: track 155.3 -> 194.8 mm, vias 0 -> 1
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- added copper zone on B.Cu, net VCC
- added copper zone on F.Cu, net VCC
