File: pcb/keyboard.kicad_sch (KiCad schematic)
At the start: 134 parts, among them J1 USB_C_Receptacle_USB2.0, J2 Programmer 1 time, J3 Addon interface, J4 Digital NOB, U1 ATmega32U4-M, Y1 16mhz

Commit message: Implement USB Hub
Other:
- sheet Bettery management and USB hub renamed USB hub
- added sheet Battery management (battery_management.kicad_sch)
- sheet USB hub: file battery_usb.kicad_sch -> usb_hub.kicad_sch
- moved on the sheet: R6

Commit message: shematic and pcb update
Parts:
- removed C10, C11, C12, C13, C14, C15, C8, C9: 100nF, Capacitor_SMD:C_0402_1005Metric, symbol Device:C
- removed C16, C17, C18, C19, C20, C21, C22, C23, C24, C25, C26, C27: 220pF, Capacitor_SMD:C_0402_1005Metric, symbol Device:C
- removed MUX1, MUX2, MUX3, MUX4, MUX5, MUX6, MUX7, MUX8: U74HC4051G-Q16, Package_DFN_QFN:QFN-16-1EP_3x3mm_P0.5mm_EP1.7x1.7mm, symbol U74HC4051G-Q16-3030-R:U74HC4051G-Q16-3030-R
- removed R10, R11, R12, R13, R14, R15, R16, R17, R18, R21, R22, R23: R10K, Resistor_SMD:R_0402_1005Metric, symbol Device:R
- removed S1, S10, S11, S12, S13, S16, S17, S18, S19, S2, S20, S21, S22, S23, S24, S25, S26, S27, S3, S30, S31, S32, S33, S34, S35, S36, S37, S38, S39, S4, S40, S43, S44, S45, S46, S47, S48, S49, S5, S50, S51, S52, S6, S60, S61, S62, S63, S64, S65, S66, S67, S7, S8, S9: PG151101S11, Button_Switch_Keyboard:SW_Cherry_MX_1.00u_PCB, symbol PG151101S11:PG151101S11
- removed S14: PG151101S11, Button_Switch_Keyboard:SW_Cherry_MX_2.00u_PCB, symbol PG151101S11:PG151101S11
- removed S15, S28: PG151101S11, Button_Switch_Keyboard:SW_Cherry_MX_1.50u_PCB, symbol PG151101S11:PG151101S11
- removed S29, S53: PG151101S11, Button_Switch_Keyboard:SW_Cherry_MX_1.75u_PCB, symbol PG151101S11:PG151101S11
- removed S41, S42: PG151101S11, Button_Switch_Keyboard:SW_Cherry_MX_2.25u_PCB, symbol PG151101S11:PG151101S11
- removed S54, S55, S56, S58, S59: PG151101S11, Button_Switch_Keyboard:SW_Cherry_MX_1.25u_PCB, symbol PG151101S11:PG151101S11
- removed S57: PG151101S11, Button_Switch_Keyboard:SW_Cherry_MX_6.25u_PCB, symbol PG151101S11:PG151101S11
Connections:
- net KEY_63_ARR_UP renamed KEY_63
- net KEY_64_ARR_LEFT renamed KEY_64
- net KEY_65_ARR_DOWN renamed KEY_65
- net KEY_66_ARR_RIGHT renamed KEY_66
Other:
- added sheet Key multiplezers (key_muxes.kicad_sch)
- added sheet Keys (keys.kicad_sch)
- note removed: "Arrow pullups"
- note removed: "Switch multiplexers"
- moved on the sheet: C1, C2, C3, C4, C5, C6, C7, D1, D2, D3, J1, J2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

Commit message: new versions and finalized wired version
Connections:
- net VIN is gone; now on net VCC: J1.A4 (VBUS), J1.A9 (VBUS), J1.B4 (VBUS), J1.B9 (VBUS)
- net LED_0: now also U1.20 (PD2); no longer U1.22 (PD5)
- net LED_2: now also U1.22 (PD5); no longer U1.20 (PD2)
Other:
- removed sheet Battery management
Changed lines of the file:
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@@
-    (effects (font (size 1.27 1.27)) (justify left bottom))
-  )
-  (label "VIN" (at 67.31 125.73 0) (fields_autoplaced)
     (effects (font (size 1.27 1.27)) (justify left bottom))
   )
@@
     (effects (font (size 1.27 1.27)) (justify left bottom))
   )
-  (label "LED_2" (at 241.3 87.63 0) (fields_autoplaced)
+  (label "LED_0" (at 241.3 87.63 0) (fields_autoplaced)
     (effects (font (size 1.27 1.27)) (justify left bottom))
   )
@@
     (effects (font (size 1.27 1.27)) (justify left bottom))
   )
+  (label "VCC" (at 71.12 125.73 180) (fields_autoplaced)
+    (effects (font (size 1.27 1.27)) (justify right bottom))
+  )
   (label "VCC" (at 243.84 41.91 0) (fields_autoplaced)
     (effects (font (size 1.27 1.27)) (justify left bottom))
@@
     (effects (font (size 1.27 1.27)) (justify left bottom))
   )
-  (label "LED_0" (at 241.3 95.25 0) (fields_autoplaced)
+  (label "LED_2" (at 241.3 95.25 0) (fields_autoplaced)
     (effects (font (size 1.27 1.27)) (justify left bottom))
   )
@@
     (instances
       (project "keyboard"
-        (path "/ba343d94-601d-44c5-b848-a7d9121c7be9" (page "5"))
+        (path "/ba343d94-601d-44c5-b848-a7d9121c7be9" (page "4"))
       )
     )
@@
       (effects (font (size 1.27 1.27)) (justify left top))
     )
-    (instances
-      (project "keyboard"
-        (path "/ba343d94-601d-44c5-b848-a7d9121c7be9" (page "4"))
-      )
-    )
-  )
-  (sheet (at -58.42 39.37) (size 39.37 22.86) (fields_autoplaced)
-    (stroke (width 0.1524) (type solid))
-    (fill (color 0 0 0 0.0000))
-    (property "Sheetname" "Battery management" (at -58.42 38.6584 0)
-      (effects (font (size 1.27 1.27)) (justify left bottom))
-    )
-    (property "Sheetfile" "battery_management.kicad_sch" (at -58.42 62.8146 0)
-      (effects (font (size 1.27 1.27)) (justify left top))
-    )
