File: kicad/default/key_muxes.kicad_sch (KiCad schematic)
At the start: 40 parts

Commit message: Add LEDs to PCB
Parts:
- renumbered C9 to C10, C13 to C11, C10 to C12, C14 to C13, C11 to C14, C20 to C17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
