File: kicad/default/keyboard.kicad_pcb (KiCad board)
At the start: 2 copper layers, 308.9 x 101.5 mm, 172 parts, among them J1 USB_C_Receptacle_USB2.0, J2 Programmer 1 time, J3 Addon interface, J4 Digital NOB, J5 USB_C1_USB2.0, J6 USB_A1, J7 USB_A2, U1 ATmega32U4-M, U2 USB2514-HZH (C184347), U3 TPS62140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

Commit message: Add LEDs to PCB
Parts:
- removed D1, D2, D3: LED, LED_THT:LED_D3.0mm_Clear
- removed R3, R4, R5: R330, Resistor_SMD:R_0402_1005Metric
- added LED0: LED, Parts:SK6812-MINI-E, B.Cu at (230.9, 137.3)
- added LED1: LED, Parts:SK6812-MINI-E, B.Cu at (254.7, 137.3)
- added LED10: LED, Parts:SK6812-MINI-E, B.Cu at (195.1, 118.3)
- added LED11: LED, Parts:SK6812-MINI-E, B.Cu at (176.1, 118.3)
- added LED12: LED, Parts:SK6812-MINI-E, B.Cu at (159.4, 137.4)
- added LED13: LED, Parts:SK6812-MINI-E, B.Cu at (157.0, 118.3)
- added LED14: LED, Parts:SK6812-MINI-E, B.Cu at (138.0, 118.3)
- added LED15: LED, Parts:SK6812-MINI-E, B.Cu at (119.0, 118.3)
- added LED16: LED, Parts:SK6812-MINI-E, B.Cu at (99.9, 118.3)
- added LED17: LED, Parts:SK6812-MINI-E, B.Cu at (80.9, 118.3)
- added LED18: LED, Parts:SK6812-MINI-E, B.Cu at (88.0, 137.4)
- added LED19: LED, Parts:SK6812-MINI-E, B.Cu at (64.2, 137.4)
- added LED2: LED, Parts:SK6812-MINI-E, B.Cu at (285.6, 137.4)
- added LED20: LED, Parts:SK6812-MINI-E, B.Cu at (40.4, 137.4)
- added LED21: LED, Parts:SK6812-MINI-E, B.Cu at (49.9, 118.3)
- added LED22: LED, Parts:SK6812-MINI-E, B.Cu at (45.0, 99.5)
- added LED23: LED, Parts:SK6812-MINI-E, B.Cu at (71.3, 99.3)
- added LED24: LED, Parts:SK6812-MINI-E, B.Cu at (90.4, 99.3)
- added LED25: LED, Parts:SK6812-MINI-E, B.Cu at (109.4, 99.3)
- added LED26: LED, Parts:SK6812-MINI-E, B.Cu at (128.4, 99.3)
- added LED27: LED, Parts:SK6812-MINI-E, B.Cu at (147.5, 99.3)
- added LED28: LED, Parts:SK6812-MINI-E, B.Cu at (166.6, 99.3)
- added LED29: LED, Parts:SK6812-MINI-E, B.Cu at (185.6, 99.3)
- added LED3: LED, Parts:SK6812-MINI-E, B.Cu at (304.6, 137.3)
- added LED30: LED, Parts:SK6812-MINI-E, B.Cu at (204.6, 99.3)
- added LED31: LED, Parts:SK6812-MINI-E, B.Cu at (223.7, 99.3)
- added LED32: LED, Parts:SK6812-MINI-E, B.Cu at (242.7, 99.3)
- added LED33: LED, Parts:SK6812-MINI-E, B.Cu at (261.8, 99.3)
- added LED34: LED, Parts:SK6812-MINI-E, B.Cu at (292.7, 99.3)
- added LED35: LED, Parts:SK6812-MINI-E, B.Cu at (299.9, 80.2)
- added LED36: LED, Parts:SK6812-MINI-E, B.Cu at (276.1, 80.2)
- added LED37: LED, Parts:SK6812-MINI-E, B.Cu at (257.0, 80.2)
- added LED38: LED, Parts:SK6812-MINI-E, B.Cu at (238.0, 80.2)
- added LED39: LED, Parts:SK6812-MINI-E, B.Cu at (219.0, 80.2)
- added LED4: LED, Parts:SK6812-MINI-E, B.Cu at (323.7, 137.4)
- added LED40: LED, Parts:SK6812-MINI-E, B.Cu at (199.9, 80.2)
- added LED41: LED, Parts:SK6812-MINI-E, B.Cu at (180.8, 80.2)
- added LED42: LED, Parts:SK6812-MINI-E, B.Cu at (161.8, 80.2)
- added LED43: LED, Parts:SK6812-MINI-E, B.Cu at (142.7, 80.2)
- added LED44: LED, Parts:SK6812-MINI-E, B.Cu at (123.7, 80.2)
- added LED45: LED, Parts:SK6812-MINI-E, B.Cu at (104.6, 80.2)
- added LED46: LED, Parts:SK6812-MINI-E, B.Cu at (85.6, 80.2)
- added LED47: LED, Parts:SK6812-MINI-E, B.Cu at (66.5, 80.2)
- added LED48: LED, Parts:SK6812-MINI-E, B.Cu at (42.7, 80.2)
- added LED49: LED, Parts:SK6812-MINI-E, B.Cu at (38.0, 61.1)
- added LED5: LED, Parts:SK6812-MINI-E, B.Cu at (304.6, 118.3)
- added LED50: LED, Parts:SK6812-MINI-E, B.Cu at (57.0, 61.1)
- added LED51: LED, Parts:SK6812-MINI-E, B.Cu at (76.1, 61.1)
- added LED52: LED, Parts:SK6812-MINI-E, B.Cu at (95.1, 61.1)
- added LED53: LED, Parts:SK6812-MINI-E, B.Cu at (114.1, 61.1)
- added LED54: LED, Parts:SK6812-MINI-E, B.Cu at (133.2, 61.1)
- added LED55: LED, Parts:SK6812-MINI-E, B.Cu at (152.2, 61.1)
- added LED56: LED, Parts:SK6812-MINI-E, B.Cu at (171.3, 61.1)
- added LED57: LED, Parts:SK6812-MINI-E, B.Cu at (190.3, 61.1)
- added LED58: LED, Parts:SK6812-MINI-E, B.Cu at (209.4, 61.1)
- added LED59: LED, Parts:SK6812-MINI-E, B.Cu at (228.4, 61.1)
- added LED6: LED, Parts:SK6812-MINI-E, B.Cu at (278.4, 118.3)
- added LED60: LED, Parts:SK6812-MINI-E, B.Cu at (247.5, 61.1)
- added LED61: LED, Parts:SK6812-MINI-E, B.Cu at (266.6, 61.1)
- added LED62: LED, Parts:SK6812-MINI-E, B.Cu at (295.1, 61.1)
- added LED63: LED, Parts:SK6812-MINI-E, B.Cu at (323.7, 61.1)
- added LED64: LED, Parts:SK6812-MINI-E, B.Cu at (323.6, 80.2)
- added LED65: LED, Parts:SK6812-MINI-E, B.Cu at (323.7, 99.3)
- added LED66: LED, Parts:SK6812-MINI-E, B.Cu at (323.7, 118.3)
- added LED7: LED, Parts:SK6812-MINI-E, B.Cu at (252.3, 118.3)
- added LED8: LED, Parts:SK6812-MINI-E, B.Cu at (233.2, 118.3)
- added LED9: LED, Parts:SK6812-MINI-E, B.Cu at (214.2, 118.3)
Connections:
- J2 pad 3: /SCL -> /SCK
- U1 pad 18: BOARD_EN -> /SCL
- U1 pad 20: /LED_0 -> unconnected-(U1-PD2-Pad20)
- U1 pad 21: /LED_1 -> LED_LIGHTS
- U1 pad 22: /LED_2 -> BOARD_EN
- U1 pad 9: /SCL -> /SCK
Routing:
- net BOARD_EN: track 355.1 -> 574.0 mm, vias 11 -> 12
- net /LED_2: track 218.0 -> 0.00 mm, vias 1 -> 0
- net LED_LIGHTS: track 0.00 -> 195.6 mm, vias 0 -> 1
- net /LED_1: track 194.8 -> 0.00 mm, vias 1 -> 0
- net unconnected-(U1-PD2-Pad20): track 0.00 -> 194.2 mm, vias 0 -> 1
- net /LED_0: track 193.5 -> 0.00 mm, vias 1 -> 0
- net KEY_66: track 168.2 -> 172.2 mm
- net KEY_65: track 133.5 -> 135.9 mm
- net KEY_64: track 122.1 -> 124.5 mm
- net KEY_63: track 140.4 -> 142.8 mm
- net KEY_19: track 38.3 -> 36.2 mm
- net KEY_23: track 38.4 -> 36.3 mm
- net KEY_05: track 65.2 -> 63.3 mm
- net KEY_04: track 49.2 -> 51.1 mm
- net KEY_03: track 53.3 -> 55.1 mm
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Other:
- board size 308.9 x 101.5 mm -> 306.9 x 97.3 mm
- board text added: "${REFERENCE}"
