File: kicad/default/keyboard.kicad_pcb (KiCad board)
At the start: 2 copper layers, 308.9 x 101.5 mm, 172 parts, among them J1 USB_C_Receptacle_USB2.0, J2 Programmer 1 time, J3 Addon interface, J4 Digital NOB, J5 USB_C1_USB2.0, J6 USB_A1, J7 USB_A2, U1 ATmega32U4-M, U2 USB2514-HZH (C184347), U3 TPS62140, U4 TPS2069C, U5 TPS2069C, U6 TPS2069C, Y1 16mhz, Y2 48mhz

Commit message: Add LEDs to PCB
Parts:
- removed D1, D2, D3: LED, LED_THT:LED_D3.0mm_Clear
- removed R3, R4, R5: R330, Resistor_SMD:R_0402_1005Metric
- added LED0: SK6812, LED_SMD:LED_SK6812_PLCC4_5.0x5.0mm_P3.2mm, F.Cu at (230.9, 138.2)
- added LED1: SK6812, LED_SMD:LED_SK6812_PLCC4_5.0x5.0mm_P3.2mm, F.Cu at (254.7, 138.2)
- added LED10: SK6812, LED_SMD:LED_SK6812_PLCC4_5.0x5.0mm_P3.2mm, F.Cu at (195.1, 119.1)
- added LED11: SK6812, LED_SMD:LED_SK6812_PLCC4_5.0x5.0mm_P3.2mm, F.Cu at (176.1, 119.1)
- added LED12: SK6812, LED_SMD:LED_SK6812_PLCC4_5.0x5.0mm_P3.2mm, F.Cu at (159.4, 138.2)
- added LED13: SK6812, LED_SMD:LED_SK6812_PLCC4_5.0x5.0mm_P3.2mm, F.Cu at (157.0, 119.2)
- added LED14: SK6812, LED_SMD:LED_SK6812_PLCC4_5.0x5.0mm_P3.2mm, F.Cu at (138.0, 119.2)
- added LED15: SK6812, LED_SMD:LED_SK6812_PLCC4_5.0x5.0mm_P3.2mm, F.Cu at (119.0, 119.2)
- added LED16: SK6812, LED_SMD:LED_SK6812_PLCC4_5.0x5.0mm_P3.2mm, F.Cu at (99.9, 119.2)
- added LED17: SK6812, LED_SMD:LED_SK6812_PLCC4_5.0x5.0mm_P3.2mm, F.Cu at (80.9, 119.2)
- added LED18: SK6812, LED_SMD:LED_SK6812_PLCC4_5.0x5.0mm_P3.2mm, F.Cu at (88.0, 138.3)
- added LED19: SK6812, LED_SMD:LED_SK6812_PLCC4_5.0x5.0mm_P3.2mm, F.Cu at (64.2, 138.2)
- added LED2: SK6812, LED_SMD:LED_SK6812_PLCC4_5.0x5.0mm_P3.2mm, F.Cu at (285.6, 138.2)
- added LED20: SK6812, LED_SMD:LED_SK6812_PLCC4_5.0x5.0mm_P3.2mm, F.Cu at (40.4, 138.2)
- added LED21: SK6812, LED_SMD:LED_SK6812_PLCC4_5.0x5.0mm_P3.2mm, F.Cu at (49.9, 119.2)
- added LED22: SK6812, LED_SMD:LED_SK6812_PLCC4_5.0x5.0mm_P3.2mm, F.Cu at (45.0, 100.3)
- added LED23: SK6812, LED_SMD:LED_SK6812_PLCC4_5.0x5.0mm_P3.2mm, F.Cu at (71.3, 100.1)
- added LED24: SK6812, LED_SMD:LED_SK6812_PLCC4_5.0x5.0mm_P3.2mm, F.Cu at (90.4, 100.1)
- added LED25: SK6812, LED_SMD:LED_SK6812_PLCC4_5.0x5.0mm_P3.2mm, F.Cu at (109.4, 100.1)
- added LED26: SK6812, LED_SMD:LED_SK6812_PLCC4_5.0x5.0mm_P3.2mm, F.Cu at (128.4, 100.1)
- added LED27: SK6812, LED_SMD:LED_SK6812_PLCC4_5.0x5.0mm_P3.2mm, F.Cu at (147.5, 100.1)
- added LED28: SK6812, LED_SMD:LED_SK6812_PLCC4_5.0x5.0mm_P3.2mm, F.Cu at (166.6, 100.1)
- added LED29: SK6812, LED_SMD:LED_SK6812_PLCC4_5.0x5.0mm_P3.2mm, F.Cu at (185.6, 100.1)
- added LED3: SK6812, LED_SMD:LED_SK6812_PLCC4_5.0x5.0mm_P3.2mm, F.Cu at (304.6, 138.2)
- added LED30: SK6812, LED_SMD:LED_SK6812_PLCC4_5.0x5.0mm_P3.2mm, F.Cu at (204.7, 100.1)
- added LED31: SK6812, LED_SMD:LED_SK6812_PLCC4_5.0x5.0mm_P3.2mm, F.Cu at (223.7, 100.1)
- added LED32: SK6812, LED_SMD:LED_SK6812_PLCC4_5.0x5.0mm_P3.2mm, F.Cu at (242.8, 100.1)
- added LED33: SK6812, LED_SMD:LED_SK6812_PLCC4_5.0x5.0mm_P3.2mm, F.Cu at (261.8, 100.1)
- added LED34: SK6812, LED_SMD:LED_SK6812_PLCC4_5.0x5.0mm_P3.2mm, F.Cu at (292.8, 100.1)
- added LED35: SK6812, LED_SMD:LED_SK6812_PLCC4_5.0x5.0mm_P3.2mm, F.Cu at (299.9, 81.0)
- added LED36: SK6812, LED_SMD:LED_SK6812_PLCC4_5.0x5.0mm_P3.2mm, F.Cu at (276.1, 81.0)
- added LED37: SK6812, LED_SMD:LED_SK6812_PLCC4_5.0x5.0mm_P3.2mm, F.Cu at (257.0, 81.0)
- added LED38: SK6812, LED_SMD:LED_SK6812_PLCC4_5.0x5.0mm_P3.2mm, F.Cu at (238.0, 81.0)
- added LED39: SK6812, LED_SMD:LED_SK6812_PLCC4_5.0x5.0mm_P3.2mm, F.Cu at (219.0, 81.0)
- added LED4: SK6812, LED_SMD:LED_SK6812_PLCC4_5.0x5.0mm_P3.2mm, F.Cu at (323.7, 138.2)
- added LED40: SK6812, LED_SMD:LED_SK6812_PLCC4_5.0x5.0mm_P3.2mm, F.Cu at (199.9, 81.0)
- added LED41: SK6812, LED_SMD:LED_SK6812_PLCC4_5.0x5.0mm_P3.2mm, F.Cu at (180.8, 81.0)
- added LED42: SK6812, LED_SMD:LED_SK6812_PLCC4_5.0x5.0mm_P3.2mm, F.Cu at (161.8, 81.0)
- added LED43: SK6812, LED_SMD:LED_SK6812_PLCC4_5.0x5.0mm_P3.2mm, F.Cu at (142.7, 81.0)
- added LED44: SK6812, LED_SMD:LED_SK6812_PLCC4_5.0x5.0mm_P3.2mm, F.Cu at (123.7, 81.0)
- added LED45: SK6812, LED_SMD:LED_SK6812_PLCC4_5.0x5.0mm_P3.2mm, F.Cu at (104.7, 81.0)
- added LED46: SK6812, LED_SMD:LED_SK6812_PLCC4_5.0x5.0mm_P3.2mm, F.Cu at (85.6, 81.0)
- added LED47: SK6812, LED_SMD:LED_SK6812_PLCC4_5.0x5.0mm_P3.2mm, F.Cu at (66.5, 81.0)
- added LED48: SK6812, LED_SMD:LED_SK6812_PLCC4_5.0x5.0mm_P3.2mm, F.Cu at (42.7, 81.0)
- added LED49: SK6812, LED_SMD:LED_SK6812_PLCC4_5.0x5.0mm_P3.2mm, F.Cu at (38.0, 62.0)
- added LED5: SK6812, LED_SMD:LED_SK6812_PLCC4_5.0x5.0mm_P3.2mm, F.Cu at (304.6, 119.1)
- added LED50: SK6812, LED_SMD:LED_SK6812_PLCC4_5.0x5.0mm_P3.2mm, F.Cu at (57.0, 62.0)
- added LED51: SK6812, LED_SMD:LED_SK6812_PLCC4_5.0x5.0mm_P3.2mm, F.Cu at (76.1, 62.0)
- added LED52: SK6812, LED_SMD:LED_SK6812_PLCC4_5.0x5.0mm_P3.2mm, F.Cu at (95.1, 62.0)
- added LED53: SK6812, LED_SMD:LED_SK6812_PLCC4_5.0x5.0mm_P3.2mm, F.Cu at (114.1, 62.0)
- added LED54: SK6812, LED_SMD:LED_SK6812_PLCC4_5.0x5.0mm_P3.2mm, F.Cu at (133.2, 62.0)
- added LED55: SK6812, LED_SMD:LED_SK6812_PLCC4_5.0x5.0mm_P3.2mm, F.Cu at (152.2, 62.0)
- added LED56: SK6812, LED_SMD:LED_SK6812_PLCC4_5.0x5.0mm_P3.2mm, F.Cu at (171.3, 62.0)
- added LED57: SK6812, LED_SMD:LED_SK6812_PLCC4_5.0x5.0mm_P3.2mm, F.Cu at (190.3, 62.0)
- added LED58: SK6812, LED_SMD:LED_SK6812_PLCC4_5.0x5.0mm_P3.2mm, F.Cu at (209.4, 62.0)
- added LED59: SK6812, LED_SMD:LED_SK6812_PLCC4_5.0x5.0mm_P3.2mm, F.Cu at (228.4, 62.0)
- added LED6: SK6812, LED_SMD:LED_SK6812_PLCC4_5.0x5.0mm_P3.2mm, F.Cu at (278.4, 119.2)
- added LED60: SK6812, LED_SMD:LED_SK6812_PLCC4_5.0x5.0mm_P3.2mm, F.Cu at (247.5, 62.0)
- added LED61: SK6812, LED_SMD:LED_SK6812_PLCC4_5.0x5.0mm_P3.2mm, F.Cu at (266.6, 62.0)
- added LED62: SK6812, LED_SMD:LED_SK6812_PLCC4_5.0x5.0mm_P3.2mm, F.Cu at (295.1, 62.0)
- added LED63: SK6812, LED_SMD:LED_SK6812_PLCC4_5.0x5.0mm_P3.2mm, F.Cu at (323.7, 62.0)
- added LED64: SK6812, LED_SMD:LED_SK6812_PLCC4_5.0x5.0mm_P3.2mm, F.Cu at (323.7, 81.0)
- added LED65: SK6812, LED_SMD:LED_SK6812_PLCC4_5.0x5.0mm_P3.2mm, F.Cu at (323.7, 100.1)
- added LED66: SK6812, LED_SMD:LED_SK6812_PLCC4_5.0x5.0mm_P3.2mm, F.Cu at (323.7, 119.1)
- added LED7: SK6812, LED_SMD:LED_SK6812_PLCC4_5.0x5.0mm_P3.2mm, F.Cu at (252.3, 119.1)
- added LED8: SK6812, LED_SMD:LED_SK6812_PLCC4_5.0x5.0mm_P3.2mm, F.Cu at (233.2, 119.1)
- added LED9: SK6812, LED_SMD:LED_SK6812_PLCC4_5.0x5.0mm_P3.2mm, F.Cu at (214.2, 119.2)
Connections:
- J2 pad 3: /SCL -> /SCK
- U1 pad 18: BOARD_EN -> /SCL
- U1 pad 20: /LED_0 -> unconnected-(U1-PD2-Pad20)
- U1 pad 21: /LED_1 -> unconnected-(U1-PD3-Pad21)
- U1 pad 22: /LED_2 -> BOARD_EN
- U1 pad 9: /SCL -> /SCK
Routing:
- net BOARD_EN: track 355.1 -> 573.1 mm, vias 11 -> 12
- net /LED_2: track 218.0 -> 0.00 mm, vias 1 -> 0
- net unconnected-(U1-PD3-Pad21): track 0.00 -> 194.8 mm, vias 0 -> 1
- net /LED_1: track 194.8 -> 0.00 mm, vias 1 -> 0
- net unconnected-(U1-PD2-Pad20): track 0.00 -> 193.5 mm, vias 0 -> 1
- net /LED_0: track 193.5 -> 0.00 mm, vias 1 -> 0
Other:
- board size 308.9 x 101.5 mm -> 306.9 x 97.3 mm
- board text added: "${REFERENCE}"
