File: kicad/default/keyboard.kicad_sch (KiCad schematic)
At the start: 27 parts, among them J1 USB_C_Receptacle_USB2.0, J2 Programmer 1 time, J3 Addon interface, J4 Digital NOB, U1 ATmega32U4-M, Y1 16mhz

Commit message: Add LEDs to PCB
Connections:
- net BOARD_EN: now also U1.22 (PD5); no longer U1.18 (PD0)
- net LED_0: no longer U1.20 (PD2)
- net LED_1: no longer U1.21 (PD3)
- net LED_2: no longer U1.22 (PD5)
- net SCL: now also U1.18 (PD0); no longer J2.3 (Pin_3), U1.9 (PB1)
- new net LED_LIGHTS: U1.21 (PD3)
- new net SCK: J2.3 (Pin_3), U1.9 (PB1)
Other:
- added sheet Leds (leds.kicad_sch)
