File: kicad/default/usb_hub.kicad_sch (KiCad schematic)
At the start: 38 parts, among them J5 USB_C1_USB2.0, J6 USB_A1, J7 USB_A2, U2 USB2514-HZH (C184347), U3 TPS62140, U4 TPS2069C, U5 TPS2069C, U6 TPS2069C, Y1 48mhz

Commit message: Add LEDs to PCB
Parts:
- renumbered C4 to C28, C4 to C29, C4 to C30, C3 to C31, C3 to C32, C1 to C33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
